Commit message: modified: meshes and urdf

File: omo_r1mini_description/urdf/omo_r1mini.urdf (robot description, URDF)
Before this commit: robot omo_r1mini, 8 links, 7 joints
Links:
- removed link caster_back_link
- added link caster_mount_link, mass 0.005; collision mesh filename=package://omo_r1mini_description/meshes/wheels/caster_wheel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 scale=1 1 1; visual mesh filename=package://omo_r1mini_description/meshes/wheels/caster_wheel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 scale=1 1 1
- added link caster_rotate_link, mass 0.005; collision mesh filename=package://omo_r1mini_description/meshes/wheels/caster_wheel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 scale=1 1 1; visual mesh filename=package://omo_r1mini_description/meshes/wheels/caster_wheel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 scale=1 1 1
- added link caster_wheel_link, mass 0.005; collision mesh filename=package://omo_r1mini_description/meshes/wheels/caster_wheel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 scale=1 1 1; visual mesh filename=package://omo_r1mini_description/meshes/wheels/caster_wheel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 scale=1 1 1
- link base_link: geometry collision mesh filename=package://omo_r1mini_description/meshes/bases/body_assy.dae scale=1 1 1; visual mesh filename=package://omo_r1mini_description/meshes/bases/body_assy.dae scale=1 1 1
- link base_scan: geometry collision mesh filename=package://omo_r1mini_description/meshes/sensors/ydlidar_ass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 scale=1 1 1; visual mesh filename=package://omo_r1mini_description/meshes/sensors/ydlidar_ass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 scale=1 1 1
- link housing_link: geometry collision mesh filename=package://omo_r1mini_description/meshes/bases/housing_body.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 scale=1 1 1; visual mesh filename=package://omo_r1mini_description/meshes/bases/housing_body.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 scale=1 1 1
- link wheel_left_link: geometry collision mesh filename=package://omo_r1mini_description/meshes/wheels/wheel_assy.d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 scale=1 1 1; visual mesh filename=package://omo_r1mini_description/meshes/wheels/wheel_assy.d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 scale=1 1 1
- link wheel_right_link: geometry collision mesh filename=package://omo_r1mini_description/meshes/wheels/wheel_assy.d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 scale=1 1 1; visual mesh filename=package://omo_r1mini_description/meshes/wheels/wheel_assy.d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 scale=1 1 1
Joints:
- removed joint caster_back_joint
- added joint caster_mount_joint: type fixed, parent base_link, child caster_mount_link, origin xyz=-0.10375 0.0 -0.00180 rpy=0 0 0
- added joint caster_rotate_joint: type fixed, parent caster_mount_link, child caster_rotate_link, origin xyz=0 0 -0.011 rpy=0 0 0
- added joint caster_wheel_joint: type fixed, parent caster_rotate_link, child caster_wheel_link, origin xyz=-0.0115 0 -0.0195 rpy=0 0 0, axis 0 1 0
- joint scan_joint: origin xyz=0 0 0.085 rpy=0 0 0 -> xyz=0 0 0.081 rpy=0 0 0
- joint wheel_left_joint: origin xyz=0 0.07 -0.018 rpy=0 0 0 -> xyz=0 0.0835 -0.01605 rpy=0 0 0
- joint wheel_right_joint: origin xyz=0 -0.07 -0.018 rpy=-3.14159265 0 0 -> xyz=0 -0.0835 -0.018 rpy=-3.14159265 0 0
